File: topeni_Arduino_Mega_Pro_Mini.brd (EAGLE design)
At the start: 13 parts

Commit message: Update wires
Parts:
- removed E$16: 220, discrete:R-7,5
- removed E$17: (no value), resistor-net:RN-5
- removed E$4: (no value), jumper:JP3Q
- removed E$9: (no value), jumper:JP1Y
- added E$1, E$7: DATA SEL, con-lstb:MA03-1
- added E$3: RF433, con-lstb:MA03-1
- added E$5: (no value), con-lstb:MA04-1
- added PROPOJKA, PROPOJKA1, PROPOJKA2, PROPOJKA3: 0, discrete:R-7,5
- moved W5100 21.0 mm to (17.8, 2.52)
- moved RELAY2 3.41 mm to (84.8, 13.5)
Routing:
- net S$57: track 0.00 -> 62.6 mm
- net S$49: track 0.00 -> 58.8 mm
- net S$45: track 0.00 -> 58.2 mm
- net S$50: track 0.00 -> 56.2 mm
- net S$51: track 0.00 -> 55.3 mm
- net S$52: track 0.00 -> 53.3 mm
- net S$53: track 0.00 -> 52.7 mm
- net S$48: track 0.00 -> 44.6 mm
- net S$69: track 0.00 -> 35.7 mm
- net S$68: track 0.00 -> 29.3 mm
- net S$46: track 0.00 -> 27.3 mm
- net S$47: track 0.00 -> 25.4 mm
- net S$38: track 29.9 -> 51.1 mm
- net S$43: track 86.0 -> 106.8 mm
- net S$37: track 15.0 -> 35.7 mm
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Other:
- board text added: "+"
- board text added: "+ 5V -"
- board text added: "-"
- board text added: "DATA"
- board text added: "RX/TX"
- board text added: "SCL / SDA / 5V / GND"
- board text added: "SCL/SDA"
- board text added: "Topeni Arduino Mega Pro Mini SIM 800L, W5100, RF433 I2C, UARD, Touch"
- board text removed: "Topeni Arduino Mega Pro Mini"

Commit message: Update Layers - fin
Parts:
- added PROPOJKA4, PROPOJKA5: 0, discrete:R-7,5
- moved E$5 11.0 mm to (86.0, 62.2)
- moved E$3 4.23 mm to (87.3, 43.2)
Routing:
- net S$73: track 0.00 -> 17.4 mm
- net S$71: track 0.00 -> 14.9 mm
- net S$74: track 0.00 -> 14.5 mm
- net S$85: track 0.00 -> 12.9 mm
- net S$83: track 0.00 -> 12.8 mm
- net S$91: track 0.00 -> 12.8 mm
- net S$81: track 0.00 -> 12.7 mm
- net S$87: track 0.00 -> 12.7 mm
- net S$89: track 0.00 -> 12.7 mm
- net S$77: track 0.00 -> 12.6 mm
- net S$66: track 8.82 -> 21.4 mm
- net S$79: track 0.00 -> 12.5 mm
- net S$67: track 13.3 -> 24.7 mm
- net S$72: track 0.00 -> 10.8 mm
- net S$75: track 0.00 -> 7.90 mm
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Other:
- board text added: "ARF/RST"
- board text added: "Topeni Arduino Mega Pro Mini SIM 800L, W5100, RF433 I2C, UART, Touch"
- board text removed: "Topeni Arduino Mega Pro Mini SIM 800L, W5100, RF433 I2C, UARD, Touch"

Commit message: Sync
Parts:
- added DIODA: D1, discrete:R-7,5
- added E$4: (no value), jumper:JP1Y
- added PROPOJKA6: 0, discrete:R-7,5
- moved W5100 23.1 mm to (17.8, 25.6)
- moved E$5 6.67 mm to (86.7, 68.8)
- moved PROPOJKA2 2.81 mm to (64.1, 38.5)
- moved PROPOJKA 2.56 mm to (61.0, 38.6)
Routing:
- net S$43: track 106.8 -> 75.1 mm
- net S$38: track 51.1 -> 27.8 mm
- net S$37: track 35.7 -> 12.6 mm
- net S$42: track 88.9 -> 73.0 mm
- net S$40: track 85.5 -> 70.5 mm
- net S$39: track 79.2 -> 64.5 mm
- net S$41: track 79.0 -> 64.3 mm
- net S$52: track 53.6 -> 68.2 mm
- net S$67: track 24.7 -> 38.1 mm
- net S$96: track 0.00 -> 13.1 mm
- net S$53: track 53.3 -> 66.1 mm
- net S$49: track 63.1 -> 75.4 mm
- net S$27: track 45.5 -> 57.2 mm
- net S$23: track 42.7 -> 54.2 mm
- net S$89: track 12.7 -> 1.20 mm
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Other:
- board text added: "5V 10 51 GND GND RESET 52 50"
- board text added: "ALARM"
- board text added: "ARF"
- board text added: "RST"
- board text removed: "ARF/RST"

Commit message: Update + sensors
Parts:
- added E$6, E$8: (no value), jumper:JP1Y
- added PROPOJKA7, PROPOJKA8: 0, discrete:R-7,5
- moved E$5 1.94 mm to (85.1, 67.8)
- moved E$3 1.00 mm to (87.5, 44.2)
- moved E$4 0.47 mm to (85.2, 57.1)
Routing:
- net S$114: track 0.00 -> 8.57 mm
- net S$113: track 0.00 -> 6.08 mm
- net S$109: track 0.00 -> 5.85 mm
- net S$112: track 0.00 -> 5.00 mm
- net S$68: track 37.6 -> 33.1 mm
- net S$67: track 38.1 -> 42.2 mm
- net S$73: track 14.7 -> 11.0 mm
- net S$49: track 75.4 -> 72.1 mm
- net S$48: track 60.5 -> 57.4 mm
- net S$110: track 0.00 -> 2.97 mm
- net S$108: track 0.00 -> 2.78 mm
- net S$72: track 8.39 -> 11.0 mm
- net S$111: track 0.00 -> 2.40 mm
- net S$104: track 4.11 -> 2.22 mm
- net S$56: track 6.79 -> 7.93 mm
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Other:
- board text added: "5V"
- board text added: "GND"
- board text added: "LAN - W5100"
- board text added: "OneWire"
- board text added: "RF433MHz"
- board text added: "SCL / - /SDA / +"
- board text added: "SIM800L EVB"
- board text removed: "SCL / SDA / 5V / GND"

Commit message: Update
Routing:
- net S$100: track 9.99 -> 11.3 mm
Changed lines of the file:
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@@
 <layer number="35" name="tGlue" color="7" fill="4" visible="no" active="yes"/>
 <layer number="36" name="bGlue" color="7" fill="5" visible="no" active="yes"/>
-<layer number="37" name="tTest" color="7" fill="1" visible="yes" active="yes"/>
-<layer number="38" name="bTest" color="7" fill="1" visible="yes" active="yes"/>
+<layer number="37" name="tTest" color="7" fill="1" visible="no" active="yes"/>
+<layer number="38" name="bTest" color="7" fill="1" visible="no" active="yes"/>
 <layer number="39" name="tKeepout" color="4" fill="11" visible="yes" active="yes"/>
 <layer number="40" name="bKeepout" color="1" fill="11" visible="yes" active="yes"/>
@@
 <signal name="S$22">
 <wire x1="79.5" y1="4.5" x2="85.47" y2="4.52" width="0.4064" layer="16"/>
-<wire x1="85.47" y1="4.52" x2="88.48" y2="7.87" width="0.4064" layer="16"/>
-<wire x1="88.48" y1="7.87" x2="90.31" y2="7.83" width="0.4064" layer="16"/>
-<wire x1="90.31" y1="7.83" x2="90.33" y2="19.85" width="0.4064" layer="16"/>
-<wire x1="90.33" y1="19.85" x2="86.21" y2="19.82" width="0.4064" layer="16"/>
+<wire x1="85.47" y1="4.52" x2="88.5" y2="7.86" width="0.4064" layer="16"/>
+<wire x1="88.5" y1="7.86" x2="90.32" y2="7.86" width="0.4064" layer="16"/>
+<wire x1="90.32" y1="7.86" x2="90.34" y2="19.82" width="0.4064" layer="16"/>
+<wire x1="90.34" y1="19.82" x2="86.21" y2="19.82" width="0.4064" layer="16"/>
 </signal>
 <signal name="S$23">
@@
 </signal>
 <signal name="S$18">
-<wire x1="47.9" y1="16.9" x2="47" y2="16" width="0.3048" layer="16"/>
-<wire x1="47" y1="16" x2="44.3" y2="16" width="0.254" layer="16"/>
-<wire x1="44.3" y1="16" x2="41.7" y2="13.4" width="0.3048" layer="16"/>
+<wire x1="47.9" y1="16.9" x2="47.04" y2="16.09" width="0.3048" layer="16"/>
+<wire x1="47.04" y1="16.09" x2="44.4" y2="16.06" width="0.3048" layer="16"/>
+<wire x1="44.4" y1="16.06" x2="41.7" y2="13.4" width="0.3048" layer="16"/>
 <wire x1="41.7" y1="13.4" x2="41.7" y2="12.5" width="0.3048" layer="16"/>
 <wire x1="41.7" y1="12.5" x2="41" y2="11.8" width="0.3048" layer="16"/>
@@
 <signal name="S$25">
 <wire x1="47.9" y1="19.4" x2="47.1" y2="18.6" width="0.3048" layer="16"/>
-<wire x1="47.1" y1="18.6" x2="44.6" y2="18.6" width="0.3048" layer="16"/>
-<wire x1="44.6" y1="18.6" x2="40.4" y2="14.4" width="0.3048" layer="16"/>
-<wire x1="40.4" y1="14.4" x2="39.9" y2="14.4" width="0.3048" layer="16"/>
+<wire x1="47.1" y1="18.6" x2="44.62" y2="18.58" width="0.3048" layer="16"/>
+<wire x1="44.62" y1="18.58" x2="39.92" y2="14.16" width="0.3048" layer="16"/>
+<wire x1="39.92" y1="14.16" x2="39.9" y2="14.4" width="0.3048" layer="16"/>
 </signal>
 <signal name="S$26">
@@
 <wire x1="23.93" y1="51.03" x2="35.46" y2="61.12" width="0.3048" layer="16"/>
 <wire x1="35.46" y1="61.12" x2="58.41" y2="61.11" width="0.3048" layer="16"/>
-<wire x1="58.41" y1="61.11" x2="58.4" y2="54.3" width="0.3048" layer="16"/>
-<wire x1="58.4" y1="54.3" x2="58.4" y2="53.6" width="0.4064" layer="16"/>
+<wire x1="58.41" y1="61.11" x2="58.4" y2="53.53" width="0.3048" layer="16"/>
 </signal>
 <signal name="S$46">
@@
 </signal>
 <signal name="S$57">
-<wire x1="90.17" y1="19.7" x2="90.34" y2="20.45" width="0.4064" layer="16"/>
+<wire x1="90.34" y1="19.71" x2="90.34" y2="20.45" width="0.4064" layer="16"/>
 <wire x1="90.34" y1="20.45" x2="90.3" y2="79.25" width="0.4064" layer="16"/>
 <wire x1="90.3" y1="79.25" x2="79.84" y2="79.24" width="0.4064" layer="16"/>
@@
 <wire x1="44.8" y1="25.03" x2="43.97" y2="24.73" width="0.254" layer="16"/>
 <wire x1="43.97" y1="24.73" x2="43.96" y2="23.8" width="0.254" layer="16"/>
-<wire x1="43.96" y1="23.8" x2="40.84" y2="20.68" width="0.254" layer="16"/>
-<wire x1="40.84" y1="20.68" x2="38.02" y2="20.68" width="0.254" layer="16"/>
+<wire x1="43.96" y1="23.8" x2="40.64" y2="20.68" width="0.254" layer="16"/>
+<wire x1="40.64" y1="20.68" x2="38.02" y2="20.68" width="0.254" layer="16"/>
 <wire x1="38.02" y1="20.68" x2="37.22" y2="19.88" width="0.254" layer="16"/>
 </signal>
@@
 <wire x1="47.48" y1="24.66" x2="46.46" y2="23.64" width="0.254" layer="16"/>
 <wire x1="46.46" y1="23.64" x2="44.83" y2="23.64" width="0.254" layer="16"/>
-<wire x1="44.83" y1="23.64" x2="40.74" y2="19.55" width="0.254" layer="16"/>
-<wire x1="40.74" y1="19.55" x2="40.16" y2="19.55" width="0.254" layer="16"/>
-<wire x1="40.16" y1="19.55" x2="40.12" y2="19.59" width="0.254" layer="16"/>
+<wire x1="44.83" y1="23.64" x2="39.98" y2="19.12" width="0.254" layer="16"/>
+<wire x1="39.98" y1="19.12" x2="39.93" y2="19.78" width="0.254" layer="16"/>
+<wire x1="39.93" y1="19.78" x2="39.5" y2="19.99" width="0.254" layer="16"/>
 </signal>
 <signal name="S$101">
-<wire x1="45.19" y1="22.45" x2="44.47" y2="22.45" width="0.254" layer="16"/>
-<wire x1="44.47" y1="22.45" x2="40.12" y2="18.1" width="0.254" layer="16"/>
-<wire x1="40.12" y1="18.1" x2="38.05" y2="18.1" width="0.254" layer="16"/>
+<wire x1="45.19" y1="22.45" x2="44.78" y2="22.45" width="0.254" layer="16"/>
+<wire x1="44.78" y1="22.45" x2="40.25" y2="18.1" width="0.254" layer="16"/>
+<wire x1="40.25" y1="18.1" x2="38.05" y2="18.1" width="0.254" layer="16"/>
 <wire x1="38.05" y1="18.1" x2="37.22" y2="17.27" width="0.254" layer="16"/>
 </signal>
@@
 <wire x1="48.05" y1="21.98" x2="47.22" y2="21.15" width="0.254" layer="16"/>
 <wire x1="47.22" y1="21.15" x2="44.72" y2="21.15" width="0.254" layer="16"/>
-<wire x1="44.72" y1="21.15" x2="40.48" y2="16.94" width="0.254" layer="16"/>
-<wire x1="40.48" y1="16.94" x2="40.05" y2="16.91" width="0.254" layer="16"/>
+<wire x1="44.72" y1="21.15" x2="40.14" y2="16.91" width="0.254" layer="16"/>
+<wire x1="40.14" y1="16.91" x2="40.05" y2="16.91" width="0.254" layer="16"/>
 </signal>
 <signal name="S$88">
@@
 </signal>
 <signal name="S$108">
-<wire x1="73.32" y1="63.07" x2="75.49" y2="63.16" width="0.4064" layer="16"/>
-<wire x1="75.49" y1="63.16" x2="75.92" y2="63.59" width="0.4064" layer="16"/>
+<wire x1="73.32" y1="63.2" x2="75.51" y2="63.18" width="0.4064" layer="16"/>
+<wire x1="75.51" y1="63.18" x2="75.92" y2="63.59" width="0.4064" layer="16"/>
 </signal>
 <signal name="S$109">
@@
 </signal>
 <signal name="S$113">
-<wire x1="73.58" y1="68.01" x2="69.95" y2="64.38" width="0.3048" layer="16"/>
-<wire x1="69.95" y1="64.38" x2="69.95" y2="63.43" width="0.3048" layer="16"/>
+<wire x1="73.58" y1="68.01" x2="69.85" y2="64.58" width="0.3048" layer="16"/>
+<wire x1="69.85" y1="64.58" x2="69.85" y2="63.63" width="0.3048" layer="16"/>
 </signal>
 <signal name="S$114">
