File: Topeni_Keypad.brd (EAGLE design)
At the start: 13 parts

Commit message: Sync
Parts:
- added E$13, E$15, E$16, E$17, E$18, E$19, E$20, E$21, E$26, E$27, E$28, E$29: (no value), discrete:R-5
- added E$22, E$23: (no value), con-lstb:MA06-1
- added E$24, E$25, E$30, E$31: (no value), jumper:JP1Y
Routing:
- net S$60: track 0.00 -> 179.1 mm
- net S$3: track 1.57 -> 109.2 mm
- net S$1: track 143.0 -> 59.6 mm
- net S$69: track 0.00 -> 65.3 mm
- net S$45: track 0.00 -> 65.2 mm
- net S$70: track 0.00 -> 63.0 mm
- net S$54: track 0.00 -> 62.1 mm
- net S$83: track 0.00 -> 60.3 mm
- net S$33: track 60.4 -> 4.49 mm
- net S$84: track 0.00 -> 55.0 mm
- net S$44: track 0.00 -> 53.2 mm
- net S$43: track 0.00 -> 52.9 mm
- net S$87: track 0.00 -> 51.0 mm
- net S$47: track 0.00 -> 49.3 mm
- net S$71: track 0.00 -> 49.2 mm
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Other:
- board text added: "5V"
- board text added: "AREF"
- board text added: "CSL/SDA"
- board text added: "RST"
- board text added: "RX/TX"

Commit message: Update + sensors
Routing:
- net S$60: track 179.1 -> 102.9 mm
- net S$23: track 1.70 -> 18.8 mm
- net S$20: track 1.48 -> 16.6 mm
- net S$17: track 1.53 -> 16.4 mm
- net S$25: track 1.66 -> 16.5 mm
- net S$29: track 1.66 -> 16.4 mm
- net S$14: track 1.70 -> 16.3 mm
- net S$27: track 1.57 -> 16.0 mm
- net S$94: track 0.00 -> 14.3 mm
- net S$8: track 1.66 -> 15.8 mm
- net S$9: track 1.97 -> 15.7 mm
- net S$10: track 2.08 -> 15.6 mm
- net S$11: track 1.84 -> 14.1 mm
- net S$56: track 14.4 -> 2.12 mm
- net S$86: track 7.95 -> 18.2 mm
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Other:
- board text added: "SDA/SCL"
- board text added: "TX/RX"
- board text removed: "CSL/SDA"
- board text removed: "RX/TX"

Commit message: Update
Routing:
- net S$22: track 1.20 -> 0.00 mm
- net S$61: track 1.99 -> 2.80 mm
Changed lines of the file:
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@@
 </signal>
 <signal name="S$65">
-<wire x1="25.86" y1="26.47" x2="25.86" y2="26.12" width="0.4064" layer="16"/>
-<wire x1="22.27" y1="26.5" x2="25.86" y2="26.47" width="0.4064" layer="16"/>
+<wire x1="24.2" y1="26.49" x2="25.31" y2="25.26" width="0.4064" layer="16"/>
+<wire x1="22.27" y1="26.5" x2="24.2" y2="26.49" width="0.4064" layer="16"/>
 </signal>
 <signal name="S$12">
@@
 </signal>
 <signal name="S$15">
-<wire x1="57.6" y1="26.6" x2="57.6" y2="25.4" width="0.4064" layer="16"/>
+<wire x1="57.45" y1="26.51" x2="57.45" y2="25.31" width="0.4064" layer="16"/>
 </signal>
 <signal name="S$16">
-<wire x1="62.7" y1="26.6" x2="62.7" y2="25.5" width="0.4064" layer="16"/>
+<wire x1="62.66" y1="26.51" x2="62.66" y2="25.41" width="0.4064" layer="16"/>
 </signal>
 <signal name="S$18">
@@
 <wire x1="31" y1="26.4" x2="31" y2="25.1" width="0.4064" layer="16"/>
 </signal>
-<signal name="S$22">
-<wire x1="25.8" y1="26.4" x2="25.8" y2="25.2" width="0.4064" layer="16"/>
-</signal>
 <signal name="S$26">
 <wire x1="73.7" y1="41.3" x2="73.7" y2="39.9" width="0.4064" layer="16"/>
@@
 <signal name="S$32">
 <wire x1="21.3" y1="-0.1" x2="21.31" y2="55.46" width="0" layer="16"/>
-<wire x1="21.31" y1="55.46" x2="97.8" y2="55.3" width="0" layer="16"/>
-<wire x1="97.8" y1="55.3" x2="97.7" y2="-0.1" width="0" layer="16"/>
+<wire x1="21.31" y1="55.46" x2="97.66" y2="55.44" width="0" layer="16"/>
+<wire x1="97.66" y1="55.44" x2="97.7" y2="-0.1" width="0" layer="16"/>
 <wire x1="97.7" y1="-0.1" x2="21.3" y2="-0.1" width="0" layer="16"/>
 </signal>
@@
 </signal>
 <signal name="S$37">
-<wire x1="82.7" y1="5.5" x2="80.5" y2="7.7" width="0.254" layer="16"/>
+<wire x1="82.79" y1="5.45" x2="80.5" y2="7.7" width="0.254" layer="16"/>
 </signal>
 <signal name="S$38">
@@
 </signal>
 <signal name="S$54">
-<wire x1="82.7" y1="15.25" x2="32.2" y2="15.25" width="0.254" layer="16"/>
+<wire x1="82.97" y1="15.25" x2="32.2" y2="15.25" width="0.254" layer="16"/>
 <wire x1="32.2" y1="15.25" x2="27.9" y2="20" width="0.254" layer="16"/>
 <wire x1="27.9" y1="20" x2="27.9" y2="21.1" width="0.254" layer="16"/>
@@
 </signal>
 <signal name="S$48">
-<wire x1="82.7" y1="20.6" x2="80.6" y2="17.47" width="0.254" layer="16"/>
+<wire x1="82.88" y1="20.75" x2="80.6" y2="17.47" width="0.254" layer="16"/>
 <wire x1="80.6" y1="17.47" x2="62.23" y2="17.47" width="0.254" layer="16"/>
 <wire x1="62.23" y1="17.47" x2="60.2" y2="19.7" width="0.254" layer="16"/>
@@
 </signal>
 <signal name="S$56">
-<wire x1="82.7" y1="23.29" x2="80.68" y2="22.66" width="0.254" layer="16"/>
+<wire x1="82.81" y1="23.33" x2="80.68" y2="22.66" width="0.254" layer="16"/>
 </signal>
 <signal name="S$57">
@@
 </signal>
 <signal name="S$61">
-<wire x1="32.96" y1="54.31" x2="32.96" y2="52.32" width="0.6096" layer="16"/>
+<wire x1="32.96" y1="54.31" x2="32.96" y2="51.51" width="0.6096" layer="16"/>
 </signal>
 <signal name="S$62">
@@
 <wire x1="93.57" y1="51.69" x2="88.37" y2="51.69" width="0.254" layer="16"/>
 <wire x1="88.37" y1="51.69" x2="86.89" y2="48.84" width="0.254" layer="16"/>
-<wire x1="86.89" y1="48.84" x2="77.74" y2="48.77" width="0.254" layer="16"/>
-<wire x1="77.74" y1="48.77" x2="76.28" y2="49.99" width="0.254" layer="16"/>
-<wire x1="76.28" y1="49.99" x2="76.27" y2="50.51" width="0.254" layer="16"/>
+<wire x1="86.89" y1="48.84" x2="77.76" y2="48.84" width="0.254" layer="16"/>
+<wire x1="77.76" y1="48.84" x2="76.32" y2="50.39" width="0.254" layer="16"/>
+<wire x1="76.32" y1="50.39" x2="76.27" y2="50.51" width="0.254" layer="16"/>
 </signal>
 <signal name="S$78">
@@
 <wire x1="87.94" y1="52.31" x2="86.3" y2="49.47" width="0.254" layer="16"/>
 <wire x1="86.3" y1="49.47" x2="84.19" y2="49.45" width="0.254" layer="16"/>
-<wire x1="84.19" y1="49.45" x2="83.2" y2="49.89" width="0.254" layer="16"/>
-<wire x1="83.2" y1="49.89" x2="83.22" y2="50.52" width="0.254" layer="16"/>
+<wire x1="84.19" y1="49.45" x2="83.24" y2="50.36" width="0.254" layer="16"/>
+<wire x1="83.24" y1="50.36" x2="83.22" y2="50.52" width="0.254" layer="16"/>
 </signal>
 <signal name="S$79">
@@
 </signal>
 <signal name="S$8">
-<wire x1="71.87" y1="7.92" x2="70.2" y2="6.25" width="0.254" layer="16"/>
+<wire x1="71.98" y1="7.99" x2="70.2" y2="6.25" width="0.254" layer="16"/>
 <wire x1="70.2" y1="6.25" x2="64.19" y2="6.22" width="0.254" layer="16"/>
 <wire x1="64.19" y1="6.22" x2="61.47" y2="7.98" width="0.254" layer="16"/>
@@
 <wire x1="57.48" y1="23.29" x2="63.16" y2="23.29" width="0.254" layer="16"/>
 <wire x1="63.16" y1="23.29" x2="63.63" y2="23.76" width="0.254" layer="16"/>
-<wire x1="63.63" y1="23.76" x2="71.69" y2="23.76" width="0.254" layer="16"/>
-<wire x1="71.69" y1="23.76" x2="72.24" y2="23.21" width="0.254" layer="16"/>
-<wire x1="72.24" y1="23.21" x2="72.24" y2="22.6" width="0.254" layer="16"/>
+<wire x1="63.63" y1="23.76" x2="71.47" y2="23.76" width="0.254" layer="16"/>
+<wire x1="71.47" y1="23.76" x2="72.25" y2="22.74" width="0.254" layer="16"/>
+<wire x1="72.25" y1="22.74" x2="72.24" y2="22.6" width="0.254" layer="16"/>
 </signal>
 <signal name="S$23">
@@
 <wire x1="57.43" y1="37.84" x2="63.16" y2="37.84" width="0.254" layer="16"/>
 <wire x1="63.16" y1="37.84" x2="63.53" y2="38.21" width="0.254" layer="16"/>
-<wire x1="63.53" y1="38.21" x2="71.63" y2="38.21" width="0.254" layer="16"/>
-<wire x1="71.63" y1="38.21" x2="72.13" y2="37.71" width="0.254" layer="16"/>
-<wire x1="72.13" y1="37.71" x2="72.13" y2="37.18" width="0.254" layer="16"/>
-</signal>
-<signal name="S$91">
-<wire x1="37.01" y1="37.92" x2="37.09" y2="37.92" width="0.254" layer="16"/>
+<wire x1="63.53" y1="38.21" x2="71.45" y2="38.21" width="0.254" layer="16"/>
+<wire x1="71.45" y1="38.21" x2="72.18" y2="37.29" width="0.254" layer="16"/>
+<wire x1="72.18" y1="37.29" x2="72.13" y2="37.16" width="0.254" layer="16"/>
 </signal>
 <signal name="S$92">

Commit message: Update
Routing:
- net S$11: track 14.1 -> 15.1 mm
- net S$41: track 36.8 -> 37.3 mm
- net S$56: track 2.23 -> 2.78 mm
- net S$75: track 2.73 -> 3.25 mm
- net S$23: track 18.8 -> 18.3 mm
