File: Topeni_Keypad.brd (EAGLE design)
At the start: 31 parts

Commit message: Update LCD
Parts:
- moved E$31 0.94 mm to (86.1, 43.2)
Routing:
- net S$95: track 0.00 -> 7.51 mm
- net S$38: track 12.6 -> 17.7 mm
- net S$40: track 28.7 -> 33.6 mm
- net S$42: track 45.1 -> 49.2 mm
- net S$45: track 65.2 -> 61.3 mm
- net S$47: track 49.3 -> 45.5 mm
- net S$55: track 33.9 -> 30.3 mm
- net S$57: track 19.2 -> 15.9 mm
- net S$34: track 4.80 -> 1.82 mm
- net S$35: track 4.84 -> 2.15 mm
- net S$53: track 1.80 -> 4.46 mm
- net S$51: track 1.85 -> 4.49 mm
- net S$49: track 7.53 -> 4.96 mm
- net S$52: track 1.84 -> 4.35 mm
- net S$36: track 4.71 -> 2.21 mm
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